File: Hardware/Bus_switch.kicad_sch (KiCad schematic)
At the start: 16 parts, among them U302 SN74CB3Q3245PWR

Commit message: V1.0
Parts:
- removed R306, R308: 10kΩ, PCM_JLCPCB:R_0603, symbol PCM_JLCPCB-Resistors:0603,10kΩ
- removed R312, R313: 0Ω, PCM_JLCPCB:R_0603, symbol PCM_JLCPCB-Resistors:0603,0Ω
Connections:
- net Chainbus.TX is gone; now on net Chainbus.SCL: R305.2
- net Chainbus.SCL: no longer R304.2
- net Chainbus.SDA: now also R304.2
- net Chainbus_In.RX: no longer names the net of U302.2 (A1)
- net Chainbus_In.TX: no longer names the net of U302.3 (A2)
- no-connect marks 1 -> 5
Other:
- note removed: "Route As Poka Yoke"
- title: MMS3 Hat template small (Change Me) -> MMS3_Hat_One_Wire
