File: Hardware/Interboard_connector.kicad_sch (KiCad schematic)
At the start: 2 parts, among them J201 Chainbus in, J202 Chainbus Out

Commit message: V1.0
Other:
- title: MMS3 Hat template small (Change Me) -> MMS3_Hat_One_Wire
Changed lines of the file:
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@@
 	(paper "A4")
 	(title_block
-		(title "MMS3 Hat template small (Change Me)")
-		(date "2077-13-75")
-		(rev "A")
+		(title "MMS3_Hat_One_Wire")
+		(date "2026-10-17")
+		(rev "V1.0")
 		(company "MiniModucard System")
 		(comment 1 "Wojciech Szafrański")
