File: Hardware/MMS3_hat_templates.kicad_sch (KiCad schematic)
At the start: 11 parts, among them U101 AMS1117

Commit message: V1.0
Other:
- removed sheet Power Connector
- sheet User Area ports: added none; removed VIN_BRD
- title: MMS3 Hat template small (Change Me) -> MMS3_Hat_One_Wire
